Commit message: modification of collision(size of base_link)

File: robots/gimbalrotor/urdf/beatle/gimbalrotor.urdf.xacro (robot description, xacro)
@@ -42,5 +42,5 @@
         <origin xyz="0 0 0" rpy="0 0 0"/>
         <geometry>
-          <box size="0.25 0.25 0.035"/>
+          <box size="0.518 0.518 0.241"/>
         </geometry>
       </collision>

Commit message: [urdf]modified urdf and mesh

File: robots/gimbalrotor/urdf/beatle/gimbalrotor.urdf.xacro (robot description, xacro)
@@ -23,18 +23,18 @@
     <link name="base_link">
       <inertial>
-        <origin xyz="-0.00598783 -0.00100288 0.07561852" rpy="0 0 0"/>
-        <mass value="2.04633752"/>
-        <inertia
-          ixx="0.05874417"
-          ixy="-0.00016819"
-          ixz="-0.00009109"
-          iyy="0.07089472"
-          iyz="-0.00009427"
-          izz="0.08695355"/>
+        <origin xyz="0.00342763 -0.00096132 0.08027425" rpy="0 0 0"/>
+        <mass value="2.12631312"/>
+        <inertia
+          ixx="0.06193652"
+          ixy="-0.00016612"
+          ixz="0.00380636"
+          iyy="0.07896117"
+          iyz="-0.00009265"
+          izz="0.09184325"/>
       </inertial>
       <visual>
         <origin xyz="0 0 0.0" rpy="0 0 0"/>
         <geometry>
-          <mesh filename="package://gimbalrotor/urdf/beatle/mesh/base_link.STL"/>
+          <mesh filename="package://gimbalrotor/urdf/beatle/mesh/base_link_withpen.STL"/>
         </geometry>
       </visual>
@@ -61,4 +61,20 @@
       <parent link="base_link"/>
       <origin rpy="0 0 0" xyz="0 0 0"/>
+      <axis xyz="0 0 1"/>
+    </joint>
+    <link name="end_effector">
+      <inertial>
+	<origin xyz="0 0 0" rpy="0 0 0"/>
+        <mass value="0.00001"/>
+        <inertia
+            ixx="0.000001" ixy="0.0" ixz="0.0"
+            iyy="0.000001" iyz="0.0"
+            izz="0.000001"/>
+      </inertial>
+    </link>
+    <joint name="base_end_effector_joint" type="fixed">
+      <child link="end_effector"/>
+      <parent link="base_link"/>
+      <origin rpy="0 0 0" xyz="0.337 0 0.195"/>
       <axis xyz="0 0 1"/>
     </joint>

Commit message: [urdf]added collision of pen-module

File: robots/gimbalrotor/urdf/beatle/gimbalrotor.urdf.xacro (robot description, xacro)
@@ -72,4 +72,10 @@
             izz="0.000001"/>
       </inertial>
+      <collision>
+        <origin xyz="0 0 0" rpy="0 0 0"/>
+        <geometry>
+          <box size="0.018 0.018 0.163"/>
+        </geometry>
+      </collision>
     </link>
     <joint name="base_end_effector_joint" type="fixed">

Commit message: [urdf]updated mass and inertia of base_link

File: robots/gimbalrotor/urdf/beatle/gimbalrotor.urdf.xacro (robot description, xacro)
@@ -23,13 +23,13 @@
     <link name="base_link">
       <inertial>
-        <origin xyz="0.00342763 -0.00096132 0.08027425" rpy="0 0 0"/>
-        <mass value="2.12631312"/>
-        <inertia
-          ixx="0.06193652"
-          ixy="-0.00016612"
-          ixz="0.00380636"
-          iyy="0.07896117"
+        <origin xyz="0.00879548 -0.00093466 0.07939277" rpy="0 0 0"/>
+        <mass value="2.18718917"/>
+        <inertia
+          ixx="0.06208193"
+          ixy="-0.00016539"
+          ixz="0.00452253"
+          iyy="0.08386063"
           iyz="-0.00009265"
-          izz="0.09184325"/>
+          izz="0.09660221"/>
       </inertial>
       <visual>

Commit message: [config][urdf]updated model and mass, inertia

File: robots/gimbalrotor/urdf/beatle/gimbalrotor.urdf.xacro (robot description, xacro)
@@ -23,13 +23,13 @@
     <link name="base_link">
       <inertial>
-        <origin xyz="0.00879548 -0.00093466 0.07939277" rpy="0 0 0"/>
-        <mass value="2.18718917"/>
-        <inertia
-          ixx="0.06208193"
-          ixy="-0.00016539"
-          ixz="0.00452253"
-          iyy="0.08386063"
-          iyz="-0.00009265"
-          izz="0.09660221"/>
+        <origin xyz="0.00859922 -0.00054638 0.08218887" rpy="0 0 0"/>
+        <mass value="2.24223241"/>
+        <inertia
+          ixx="0.06463170"
+          ixy="-0.00016812"
+          ixz="0.00453111"
+          iyy="0.08594030"
+          iyz="0.00005885"
+          izz="0.09711048"/>
       </inertial>
       <visual>
