Commit message: [gimbalrotor/urdf](gimbalrotor_camera_sim.urdf.xacro)dummy links for collision judge

File: robots/gimbalrotor/urdf/beatle/gimbalrotor_camera_sim.urdf.xacro (robot description, xacro)
@@ -2,4 +2,27 @@
 <robot
     xmlns:xacro="http://www.ros.org/wiki/xacro" name="gimbalrotor_link" >
+  <xacro:macro name="dummy_collision_link" params="name parent s_xyz o_xyz rpy j_xyz j_rpy">
+    <link name="${name}">
+      <inertial>
+        <origin xyz="0 0 0" rpy="0 0 0"/>
+        <mass value="0.00001"/>
+        <inertia
+            ixx="0.000001" ixy="0.0" ixz="0.0"
+            iyy="0.000001" iyz="0.0"
+            izz="0.000001"/>
+      </inertial>
+      <collision>
+        <origin xyz="${o_xyz}" rpy="${rpy}"/>
+        <geometry>
+          <box size="${s_xyz}"/>
+        </geometry>
+      </collision>
+    </link>
+    <joint name="${name}_joint" type="fixed">
+      <parent link="${parent}"/>
+      <child link="${name}"/>
+      <origin xyz="${j_xyz}" rpy="${j_rpy}"/>
+    </joint>
+  </xacro:macro>
   <xacro:macro name="gimbalrotor_center_link" params="child1 child2 child3 child4">
     ## dummy
@@ -74,7 +97,7 @@
       </inertial>
       <collision>
-        <origin xyz="0 0 0" rpy="0 0 0"/>
-        <geometry>
-          <box size="0.018 0.018 0.163"/>
+        <origin xyz="-0.0815 0 0" rpy="0 0 0"/>
+        <geometry>
+          <box size="0.163 0.018 0.018"/>
         </geometry>
       </collision>
@@ -86,4 +109,9 @@
       <axis xyz="0 0 1"/>
     </joint>
+    ## collision roller
+    <xacro:dummy_collision_link name="col_roller_up_left" parent="base_link" s_xyz="0.084 0.01 0.01" o_xyz="-0.042 0 0" rpy="0 0 0" j_xyz="0.332 -0.06 0.239" j_rpy="0 0 0"/>
+    <xacro:dummy_collision_link name="col_roller_up_right" parent="base_link" s_xyz="0.084 0.01 0.01" o_xyz="-0.042 0 0" rpy="0 0 0" j_xyz="0.332 0.06 0.239" j_rpy="0 0 0"/>
+    <xacro:dummy_collision_link name="col_roller_bottom_left" parent="base_link" s_xyz="0.084 0.01 0.01" o_xyz="-0.042 0 0" rpy="0 0 0" j_xyz="0.332 -0.06 0.003" j_rpy="0 0 0"/>
+    <xacro:dummy_collision_link name="col_roller_bottom_right" parent="base_link" s_xyz="0.084 0.01 0.01" o_xyz="-0.042 0 0" rpy="0 0 0" j_xyz="0.332 0.06 0.003" j_rpy="0 0 0"/>
     ## camera
     <link name="aerial_robot_camera_frame">

Commit message: [gimbalrotor/urdf]collision of roller(friction coefficient, slip)

File: robots/gimbalrotor/urdf/beatle/gimbalrotor_camera_sim.urdf.xacro (robot description, xacro)
@@ -2,5 +2,5 @@
 <robot
     xmlns:xacro="http://www.ros.org/wiki/xacro" name="gimbalrotor_link" >
-  <xacro:macro name="dummy_collision_link" params="name parent s_xyz o_xyz rpy j_xyz j_rpy">
+  <xacro:macro name="dummy_collision_link" params="name parent r o_xyz rpy j_xyz j_rpy">
     <link name="${name}">
       <inertial>
@@ -15,5 +15,6 @@
         <origin xyz="${o_xyz}" rpy="${rpy}"/>
         <geometry>
-          <box size="${s_xyz}"/>
+          <!-- <box size="${s_xyz}"/> -->
+	  <sphere radius="${r}"/>
         </geometry>
       </collision>
@@ -24,4 +25,10 @@
       <origin xyz="${j_xyz}" rpy="${j_rpy}"/>
     </joint>
+    <gazebo reference="${name}">
+      <mu1>0.01</mu1>
+      <mu2>0.01</mu2>
+      <slip1>0.1</slip1>
+      <slip2>0.1</slip2>
+    </gazebo>
   </xacro:macro>
   <xacro:macro name="gimbalrotor_center_link" params="child1 child2 child3 child4">
@@ -110,8 +117,12 @@
     </joint>
     ## collision roller
-    <xacro:dummy_collision_link name="col_roller_up_left" parent="base_link" s_xyz="0.084 0.01 0.01" o_xyz="-0.042 0 0" rpy="0 0 0" j_xyz="0.332 -0.06 0.239" j_rpy="0 0 0"/>
-    <xacro:dummy_collision_link name="col_roller_up_right" parent="base_link" s_xyz="0.084 0.01 0.01" o_xyz="-0.042 0 0" rpy="0 0 0" j_xyz="0.332 0.06 0.239" j_rpy="0 0 0"/>
-    <xacro:dummy_collision_link name="col_roller_bottom_left" parent="base_link" s_xyz="0.084 0.01 0.01" o_xyz="-0.042 0 0" rpy="0 0 0" j_xyz="0.332 -0.06 0.003" j_rpy="0 0 0"/>
-    <xacro:dummy_collision_link name="col_roller_bottom_right" parent="base_link" s_xyz="0.084 0.01 0.01" o_xyz="-0.042 0 0" rpy="0 0 0" j_xyz="0.332 0.06 0.003" j_rpy="0 0 0"/>
+    <!-- <xacro:dummy_collision_link name="col_roller_up_left" parent="base_link" s_xyz="0.084 0.01 0.01" o_xyz="-0.042 0 0" rpy="0 0 0" j_xyz="0.332 -0.06 0.239" j_rpy="0 0 0"/> -->
+    <!-- <xacro:dummy_collision_link name="col_roller_up_right" parent="base_link" s_xyz="0.084 0.01 0.01" o_xyz="-0.042 0 0" rpy="0 0 0" j_xyz="0.332 0.06 0.239" j_rpy="0 0 0"/> -->
+    <!-- <xacro:dummy_collision_link name="col_roller_bottom_left" parent="base_link" s_xyz="0.084 0.01 0.01" o_xyz="-0.042 0 0" rpy="0 0 0" j_xyz="0.332 -0.06 0.003" j_rpy="0 0 0"/> -->
+    <!-- <xacro:dummy_collision_link name="col_roller_bottom_right" parent="base_link" s_xyz="0.084 0.01 0.01" o_xyz="-0.042 0 0" rpy="0 0 0" j_xyz="0.332 0.06 0.003" j_rpy="0 0 0"/> -->
+    <xacro:dummy_collision_link name="col_roller_up_left" parent="base_link" r="0.005" o_xyz="0 0 0" rpy="0 0 0" j_xyz="0.332 -0.06 0.239" j_rpy="0 0 0"/>
+    <xacro:dummy_collision_link name="col_roller_up_right" parent="base_link" r="0.005" o_xyz="0 0 0" rpy="0 0 0" j_xyz="0.332 0.06 0.239" j_rpy="0 0 0"/>
+    <xacro:dummy_collision_link name="col_roller_bottom_left" parent="base_link" r="0.005" o_xyz="0 0 0" rpy="0 0 0" j_xyz="0.332 -0.06 0.003" j_rpy="0 0 0"/>
+    <xacro:dummy_collision_link name="col_roller_bottom_right" parent="base_link" r="0.005" o_xyz="0 0 0" rpy="0 0 0" j_xyz="0.332 0.06 0.003" j_rpy="0 0 0"/>
     ## camera
     <link name="aerial_robot_camera_frame">
