Commit message: [camera] update hole_deviation_compensator.py (recovery when detection fails), hole_world_estimate_compensator.py (estimation of hole position in world frame)

File: robots/gimbalrotor/urdf/beatle/gimbalrotor_camera_sim.urdf.xacro (robot description, xacro)
@@ -146,5 +146,5 @@
       <parent link="base_link"/>
       <child link="aerial_robot_camera_frame"/>
-      <origin xyz="0.259 0 0.159" rpy="0 ${-pi/6} 0"/>
+      <origin xyz="0.259 0 0.159" rpy="0 ${-pi/9} 0"/>
     </joint>
     ## camera optical frame
