Commit message: [gimbalrotor] update urdf of beatle (mass and inertia)

File: robots/gimbalrotor/urdf/beatle/gimbalrotor_attachment_roller.urdf.xacro (robot description, xacro)
@@ -23,13 +23,13 @@
     <link name="base_link">
       <inertial>
-        <origin xyz="0.01245780 -0.00024510 0.08607289" rpy="0 0 0"/>
-        <mass value="2.31523483"/>
-        <inertia
-          ixx="0.06815349"
-          ixy="-0.00000680"
-          ixz="0.00693414"
-          iyy="0.09316127"
-          iyz="0.00016826"
-          izz="0.10154939"/>
+        <origin xyz="0.02920179 0.00202296 0.09409091" rpy="0 0 0"/>
+        <mass value="2.48383571"/>
+        <inertia
+          ixx="0.07588224"
+          ixy="0.00136943"
+          ixz="0.01587034"
+          iyy="0.11140947"
+          iyz="0.00130753"
+          izz="0.11413637"/>
       </inertial>
       <visual>

Commit message: [gimbalrotor] change endeffector position, update get_tf.py (high-frequency topic publishing)

File: robots/gimbalrotor/urdf/beatle/gimbalrotor_attachment_roller.urdf.xacro (robot description, xacro)
@@ -83,5 +83,5 @@
       <child link="end_effector"/>
       <parent link="base_link"/>
-      <origin rpy="0 0 0" xyz="0.337 0 0.195"/>
+      <origin rpy="0 0 0" xyz="0.331 0 0.204"/>
       <axis xyz="0 0 1"/>
     </joint>
