Commit message: [aerial_robot_model.launch, gimbalrotor] on/off simulation camera

File: robots/gimbalrotor/robots/beatle/gimbalrotor.gazebo.xacro (robot description, xacro)
@@ -3,4 +3,6 @@
     xmlns:xacro="http://www.ros.org/wiki/xacro" name="gimbalrotor" >
   <xacro:arg name="robot_name" default="gimbalrotor" />
+  <xacro:arg name="enable_camera" default="false" />
+  <xacro:property name="enable_camera" value="$(arg enable_camera)"/>
   <!-- <xacro:include filename="$(find gimbalrotor)/robots/beatle/gimbalrotor.urdf.xacro" /> -->
   <xacro:include filename="$(find gimbalrotor)/robots/beatle/gimbalrotor_camera_sim.urdf.xacro" />
@@ -8,38 +10,40 @@
   <xacro:include filename="$(find aerial_robot_simulation)/xacro/spinal.gazebo.xacro" />
   <xacro:gazebo_spinal robot_name="$(arg robot_name)" mag_frame="fc" />
-  <gazebo reference="aerial_robot_camera_frame">
-    <sensor type="camera" name="aerial_robot_camera">
-      <update_rate>30.0</update_rate>
-      <camera name="head">
-	<horizontal_fov>1.57</horizontal_fov>
-	<image>
-          <width>1280</width>
-          <height>720</height>
-          <format>RGB</format>
-	</image>
-	<clip>
-          <near>0.02</near>
-          <far>300</far>
-	</clip>
-	<noise>
-          <type>gaussian</type>
-          <mean>0.0</mean>
-          <stddev>0.007</stddev>
-	</noise>
-      </camera>
-      <plugin name="camera_controller" filename="libgazebo_ros_camera.so">
-	<robotNamespace>/$(arg robot_name)</robotNamespace>
-	<cameraName>usb_cam</cameraName>
-	<imageTopicName>image_raw</imageTopicName>
-	<cameraInfoTopicName>camera_info</cameraInfoTopicName>
-	<frameName>$(arg robot_name)/aerial_robot_camera_optical_frame</frameName>
-	<hackBaseline>0.07</hackBaseline>
-	<distortionK1>0.0</distortionK1>
-	<distortionK2>0.0</distortionK2>
-	<distortionK3>0.0</distortionK3>
-	<distortionT1>0.0</distortionT1>
-	<distortionT2>0.0</distortionT2>
-      </plugin>
-    </sensor>
-  </gazebo>
+  <xacro:if value="${enable_camera}">
+    <gazebo reference="aerial_robot_camera_frame">
+      <sensor type="camera" name="aerial_robot_camera">
+	<update_rate>30.0</update_rate>
+	<camera name="head">
+	  <horizontal_fov>1.57</horizontal_fov>
+	  <image>
+            <width>1280</width>
+            <height>720</height>
+            <format>RGB</format>
+	  </image>
+	  <clip>
+            <near>0.02</near>
+            <far>300</far>
+	  </clip>
+	  <noise>
+            <type>gaussian</type>
+            <mean>0.0</mean>
+            <stddev>0.007</stddev>
+	  </noise>
+	</camera>
+	<plugin name="camera_controller" filename="libgazebo_ros_camera.so">
+	  <robotNamespace>/$(arg robot_name)</robotNamespace>
+	  <cameraName>usb_cam</cameraName>
+	  <imageTopicName>image_raw</imageTopicName>
+	  <cameraInfoTopicName>camera_info</cameraInfoTopicName>
+	  <frameName>$(arg robot_name)/aerial_robot_camera_optical_frame</frameName>
+	  <hackBaseline>0.07</hackBaseline>
+	  <distortionK1>0.0</distortionK1>
+	  <distortionK2>0.0</distortionK2>
+	  <distortionK3>0.0</distortionK3>
+	  <distortionT1>0.0</distortionT1>
+	  <distortionT2>0.0</distortionT2>
+	</plugin>
+      </sensor>
+    </gazebo>
+  </xacro:if>
 </robot>

File: robots/gimbalrotor/robots/beatle/gimbalrotor_camera_sim.urdf.xacro (robot description, xacro)
@@ -2,4 +2,5 @@
 <robot
     xmlns:xacro="http://www.ros.org/wiki/xacro" name="gimbalrotor" >
+  <xacro:arg name="enable_camera" default="false" />
   <xacro:include filename="$(find gimbalrotor)/urdf/beatle/gimbalrotor_camera_sim.urdf.xacro" />
   <!-- <xacro:include filename="$(find gimbalrotor)/urdf/beatle/gimbalrotor_attachment.urdf.xacro" /> -->

File: robots/gimbalrotor/urdf/beatle/gimbalrotor_camera_sim.urdf.xacro (robot description, xacro)
@@ -2,4 +2,5 @@
 <robot
     xmlns:xacro="http://www.ros.org/wiki/xacro" name="gimbalrotor_link" >
+  <xacro:property name="enable_camera" default="false" />
   <xacro:macro name="dummy_collision_link" params="name parent r o_xyz rpy j_xyz j_rpy">
     <link name="${name}">

Commit message: [camera][gimbalrotor] simulation environment for extruding exp & others

File: robots/gimbalrotor/robots/beatle/gimbalrotor.gazebo.xacro (robot description, xacro)
@@ -47,3 +47,16 @@
     </gazebo>
   </xacro:if>
+  <!-- <gazebo reference="base_link"> -->
+  <!--   <visual> -->
+  <!--     <plugin name="trajectory_visual_plugin" -->
+  <!--             filename="libtrajectory_visual_plugin.so"/> -->
+  <!--   </visual> -->
+  <!-- </gazebo> -->
+  <!-- <gazebo reference="base_link"> -->
+  <!--   <visual> -->
+  <!--     <plugin name="trajectory_visualizer" filename="libtrajectory_visualizer.so"> -->
+  <!-- 	<pose_topic>/gimbalrotor/endeffector_pose</pose_topic> -->
+  <!--     </plugin> -->
+  <!--   </visual> -->
+  <!-- </gazebo> -->
 </robot>
